File: 12Vbuck.kicad_sch (KiCad schematic)
At the start: 32 parts, among them Q1 NMOS, Q2 NMOS, U1 LM5146RGYR

Commit message: endring av kondensatorer
Parts:
- added R311: 20k, symbol Device:R
- C311: Field5 C_In3 -> C_In2
- C312: Field5 C_In2 -> C_In3
- C314: value 22u -> 1u
- C315, C316: value 22u -> 10u
- C317, C318: value 22u -> 47u
- L301: value L -> 6.8u
- R308: Field5 R_FB1 -> R_FB2
- R309: value 100k -> 21k; Field5 R_C2 -> R_FB1
- R310: value 21k -> 100k; Field5 R_FB1 -> R_C2
Connections:
- net 12VV_out is gone; now on net 12V_Vout: C314.1, L301.2, R309.1, R310.2
- net 12V_Vin: now also C310.1, C311.1, C312.1, C313.1
- net GND: no longer C313.2, C318.2, Q2.3 (S), U1.12 (PGND)
- net 12V_Vout: now reaches C318.1
- net 12V_Vout: now also C315.1, C316.1, C317.1; no longer C317.2
- net V_cc: now reaches C303.1, U1.14 (VCC)
- net V_cc: now also R311.2
- net PGND: now reaches C316.2
- net PGND: now also C309.2, C310.2, C311.2, C312.2, C313.2, C314.2, C315.2, C317.2, C318.2; no longer C317.1
- net at C305.1, R306.1, U1.11 (ILIM): now also R311.1
- new net: Q2.3 (S), U1.12 (PGND)
Other:
- moved on the sheet: C303, C306, C307, C308, C309, C310, C311, C312, C313, C314, C315, C316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

Commit message: fant 1 komp:)
Parts:
- C317, C318: footprint (none) -> CAPAE830X1000N; symbol Device:C -> Halfdan:APA0809470M050R; Height (none) -> 10; Manufacturer_Name (none) -> Kyocera AVX; Manufacturer_Part_Number (none) -> APA0809470M050R; Mouser Part Number (none) -> 581-APA0809470M050R; Mouser Price/Stock (none) -> https://www.mouser.co.uk/ProductDetail/KYOCERA-AVX/APA08094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
Connections:
- net 12V_Vout: now also C317.2 (-), C318.2 (-); no longer C317.1, C318.1
- net PGND: now also C317.1 (+), C318.1 (+); no longer C317.2, C318.2
Changed lines of the file:
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@@
 	)
 	(junction
-		(at 220.98 91.44)
-		(diameter 0)
-		(color 0 0 0 0)
-	)
-	(junction
 		(at 220.98 72.39)
 		(diameter 0)
@@
 	)
 	(junction
+		(at 223.52 104.14)
+		(diameter 0)
+		(color 0 0 0 0)
+	)
+	(junction
 		(at 198.12 99.06)
 		(diameter 0)
@@
 	)
 	(junction
-		(at 260.35 110.49)
+		(at 209.55 104.14)
 		(diameter 0)
 		(color 0 0 0 0)
 	)
 	(junction
-		(at 220.98 99.06)
+		(at 260.35 110.49)
 		(diameter 0)
 		(color 0 0 0 0)
@@
 	)
 	(junction
+		(at 223.52 91.44)
+		(diameter 0)
+		(color 0 0 0 0)
+	)
+	(junction
 		(at 102.87 72.39)
 		(diameter 0)
@@
 	(wire
 		(pts
-			(xy 209.55 99.06) (xy 209.55 102.87)
+			(xy 209.55 99.06) (xy 209.55 104.14)
 		)
 		(stroke
@@
 	(wire
 		(pts
-			(xy 220.98 91.44) (xy 232.41 91.44)
-		)
-		(stroke
-			(width 0)
-			(type default)
-		)
-	)
-	(wire
-		(pts
 			(xy 186.69 80.01) (xy 198.12 80.01)
 		)
@@
 	(wire
 		(pts
-			(xy 209.55 99.06) (xy 220.98 99.06)
+			(xy 209.55 104.14) (xy 232.41 104.14)
 		)
 		(stroke
@@
 	(wire
 		(pts
-			(xy 209.55 91.44) (xy 220.98 91.44)
+			(xy 209.55 91.44) (xy 232.41 91.44)
 		)
 		(stroke
@@
 	(wire
 		(pts
-			(xy 220.98 99.06) (xy 232.41 99.06)
-		)
-		(stroke
-			(width 0)
-			(type default)
-		)
-	)
-	(wire
-		(pts
 			(xy 167.64 100.33) (xy 167.64 101.6)
 		)
@@
 	)
 	(symbol
-		(lib_id "Device:C")
-		(at 232.41 95.25 0)
+		(lib_id "Halfdan:APA0809470M050R")
+		(at 232.41 104.14 90)
 		(unit 1)
 		(body_style 1)
@@
 		(dnp no)
 		(property "Reference" "C318"
-			(at 236.22 93.9799 0)
+			(at 231.1399 100.33 0)
 			(show_name no)
 			(do_not_autoplace no)
@@
 		)
 		(property "Value" "47u"
-			(at 236.22 96.5199 0)
+			(at 233.6799 100.33 0)
 			(show_name no)
 			(do_not_autoplace no)
@@
 			)
 		)
-		(property "Footprint" ""
-			(at 233.3752 99.06 0)
+		(property "Footprint" "CAPAE830X1000N"
+			(at 328.6 95.25 0)
 			(hide yes)
 			(show_name no)
@@
 					(size 1.27 1.27)
 				)
+				(justify left top)
 			)
 		)
-		(property "Datasheet" ""
-			(at 232.41 95.25 0)
+		(property "Datasheet" "https://datasheets.kyocera-avx.com/kyocera-avx-apa-series.pdf"
+			(at 428.6 95.25 0)
 			(hide yes)
 			(show_name no)
@@
 					(size 1.27 1.27)
 				)
+				(justify left top)
 			)
 		)
-		(property "Description" "Unpolarized capacitor"
-			(at 232.41 95.25 0)
+		(property "Description" "Aluminum Organic Polymer Capacitors 47UF       50V"
+			(at 232.41 104.14 0)
 			(hide yes)
 			(show_name no)
@@
 		)
 		(property "Field5" "C_Out1"
-			(at 238.252 98.806 0)
+			(at 235.966 98.298 0)
+			(show_name no)
+			(do_not_autoplace no)
+			(effects
+				(font
+					(size 1.27 1.27)
+				)
+			)
+		)
+		(property "Height" "10"
+			(at 628.6 95.25 0)
+			(hide yes)
+			(show_name no)
+			(do_not_autoplace no)
+			(effects
+				(font
+					(size 1.27 1.27)
+				)
+				(justify left top)
+			)
+		)
+		(property "Mouser Part Number" "581-APA0809470M050R"
+			(at 728.6 95.25 0)
+			(hide yes)
+			(show_name no)
+			(do_not_autoplace no)
+			(effects
+				(font
+					(size 1.27 1.27)
+				)
+				(justify left top)
+			)
+		)
+		(property "Mouser Price/Stock" "https://www.mouser.co.uk/ProductDetail/KYOCERA-AVX/APA0809470M050R?qs=Wj%2FVkw3K%252BMAkqelysx9Hrg%3D%3D"
+			(at 828.6 95.25 0)
+			(hide yes)
+			(show_name no)
+			(do_not_autoplace no)
+			(effects
+				(font
+					(size 1.27 1.27)
+				)
+				(justify left top)
+			)
+		)
+		(property "Manufacturer_Name" "Kyocera AVX"
+			(at 928.6 95.25 0)
+			(hide yes)
 			(show_name no)
 			(do_not_autoplace no)
@@
 					(size 1.27 1.27)
 				)
+				(justify left top)
+			)
+		)
+		(property "Manufacturer_Part_Number" "APA0809470M050R"
+			(at 1028.6 95.25 0)
+			(hide yes)
+			(show_name no)
+			(do_not_autoplace no)
+			(effects
+				(font
+					(size 1.27 1.27)
+				)
+				(justify left top)
 			)
 		)
@@
 	)
 	(symbol
-		(lib_id "Device:C")
-		(at 220.98 95.25 0)
+		(lib_id "Halfdan:APA0809470M050R")
+		(at 223.52 104.14 90)
 		(unit 1)
 		(body_style 1)
@@
 		(dnp no)
 		(property "Reference" "C317"
-			(at 224.79 93.9799 0)
+			(at 222.2499 100.33 0)
 			(show_name no)
 			(do_not_autoplace no)
@@
 		)
 		(property "Value" "47u"
-			(at 224.79 96.5199 0)
+			(at 224.7899 100.33 0)
 			(show_name no)
 			(do_not_autoplace no)
@@
 			)
 		)
-		(property "Footprint" ""
-			(at 221.9452 99.06 0)
+		(property "Footprint" "CAPAE830X1000N"
+			(at 319.71 95.25 0)
 			(hide yes)
 			(show_name no)
@@
 					(size 1.27 1.27)
 				)
+				(justify left top)
 			)
 		)
-		(property "Datasheet" ""
-			(at 220.98 95.25 0)
+		(property "Datasheet" "https://datasheets.kyocera-avx.com/kyocera-avx-apa-series.pdf"
+			(at 419.71 95.25 0)
 			(hide yes)
 			(show_name no)
@@
 					(size 1.27 1.27)
 				)
+				(justify left top)
 			)
 		)
-		(property "Description" "Unpolarized capacitor"
-			(at 220.98 95.25 0)
+		(property "Description" "Aluminum Organic Polymer Capacitors 47UF       50V"
+			(at 223.52 104.14 0)
 			(hide yes)
 			(show_name no)
@@
 		)
 		(property "Field5" "C_Out2"
-			(at 227.33 98.298 0)
+			(at 226.568 97.79 0)
+			(show_name no)
+			(do_not_autoplace no)
+			(effects
+				(font
+					(size 1.27 1.27)
+				)
+			)
+		)
+		(property "Height" "10"
+			(at 619.71 95.25 0)
+			(hide yes)
 			(show_name no)
 			(do_not_autoplace no)
@@
 					(size 1.27 1.27)
 				)
+				(justify left top)
+			)
+		)
+		(property "Mouser Part Number" "581-APA0809470M050R"
+			(at 719.71 95.25 0)
+			(hide yes)
+			(show_name no)
+			(do_not_autoplace no)
+			(effects
+				(font
+					(size 1.27 1.27)
+				)
+				(justify left top)
+			)
+		)
+		(property "Mouser Price/Stock" "https://www.mouser.co.uk/ProductDetail/KYOCERA-AVX/APA0809470M050R?qs=Wj%2FVkw3K%252BMAkqelysx9Hrg%3D%3D"
+			(at 819.71 95.25 0)
+			(hide yes)
+			(show_name no)
+			(do_not_autoplace no)
+			(effects
+				(font
+					(size 1.27 1.27)
+				)
+				(justify left top)
+			)
+		)
+		(property "Manufacturer_Name" "Kyocera AVX"
+			(at 919.71 95.25 0)
+			(hide yes)
+			(show_name no)
+			(do_not_autoplace no)
+			(effects
+				(font
+					(size 1.27 1.27)
+				)
+				(justify left top)
+			)
+		)
+		(property "Manufacturer_Part_Number" "APA0809470M050R"
+			(at 1019.71 95.25 0)
+			(hide yes)
+			(show_name no)
+			(do_not_autoplace no)
+			(effects
+				(font
+					(size 1.27 1.27)
+				)
+				(justify left top)
 			)
 		)
@@
 	(symbol
 		(lib_id "power:GND")
-		(at 209.55 102.87 0)
+		(at 209.55 104.14 0)
 		(unit 1)
 		(body_style 1)
@@
 		(fields_autoplaced yes)
 		(property "Reference" "#PWR019"
-			(at 209.55 109.22 0)
+			(at 209.55 110.49 0)
 			(hide yes)
 			(show_name no)
@@
 		)
 		(property "Value" "PGND"
-			(at 209.55 107.95 0)
+			(at 209.55 109.22 0)
 			(show_name no)
 			(do_not_autoplace no)
@@
 		)
 		(property "Footprint" ""
-			(at 209.55 102.87 0)
+			(at 209.55 104.14 0)
 			(hide yes)
 			(show_name no)
@@
 		)
 		(property "Datasheet" ""
-			(at 209.55 102.87 0)
+			(at 209.55 104.14 0)
 			(hide yes)
 			(show_name no)
@@
 		)
 		(property "Description" "Power symbol creates a global label with name \"GND\" , ground"
-			(at 209.55 102.87 0)
+			(at 209.55 104.14 0)
 			(hide yes)
 			(show_name no)
