File: ProteusPowerManagment.kicad_sch (KiCad schematic)
At the start: 0 parts

Commit message: Fysiske komp for 24V
Other:
- sheet 24Vbuck ports: added 24VPGOOD, 24V_VINN, 24V_VOUT, 24Vsync_inn, 24Vsync_out; removed none
Changed lines of the file:
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@@
+			)
+		)
+		(pin "24VPGOOD" output
+			(at 78.74 43.18 0)
+			(effects
+				(font
+					(size 1.27 1.27)
+				)
+				(justify right)
+			)
+		)
+		(pin "24Vsync_inn" input
+			(at 39.37 43.18 180)
+			(effects
+				(font
+					(size 1.27 1.27)
+				)
+				(justify left)
+			)
+		)
+		(pin "24Vsync_out" output
+			(at 78.74 45.72 0)
+			(effects
+				(font
+					(size 1.27 1.27)
+				)
+				(justify right)
+			)
+		)
+		(pin "24V_VOUT" output
+			(at 78.74 49.53 0)
+			(effects
+				(font
+					(size 1.27 1.27)
+				)
+				(justify right)
+			)
+		)
+		(pin "24V_VINN" input
+			(at 39.37 46.99 180)
+			(effects
+				(font
+					(size 1.27 1.27)
+				)
+				(justify left)
 			)
 		)
