File: ProteusPowerManagment.kicad_sch (KiCad schematic)
At the start: 0 parts

Commit message: try again
Other:
- added sheet 12Vbuck (12Vbuck.kicad_sch)
- added sheet 24Vbuck (24Vbuck.kicad_sch)
- added sheet 5Vbuck (5Vbuck.kicad_sch)
Changed lines of the file:
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@@
 	(generator_version "10.0")
 	(paper "A4")
+	(sheet
+		(at 39.37 39.37)
+		(size 39.37 33.02)
+		(exclude_from_sim no)
+		(in_bom yes)
+		(on_board yes)
+		(dnp no)
+		(fields_autoplaced yes)
+		(stroke
+			(width 0.1524)
+			(type solid)
+		)
+		(fill
+			(color 0 0 0 0)
+		)
+		(property "Sheetname" "24Vbuck"
+			(at 39.37 38.6584 0)
+			(show_name no)
+			(do_not_autoplace no)
+			(effects
+				(font
+					(size 1.27 1.27)
+				)
+				(justify left bottom)
+			)
+		)
+		(property "Sheetfile" "24Vbuck.kicad_sch"
+			(at 39.37 72.9746 0)
+			(show_name no)
+			(do_not_autoplace no)
+			(effects
+				(font
+					(size 1.27 1.27)
+				)
+				(justify left top)
+			)
+		)
+		(instances
+			(project "ProteusPowerManagment"
+				(path "/c24111dd-5300-4143-a3c3-2d963194a3cb"
+					(page "2")
+				)
+			)
+		)
+	)
+	(sheet
+		(at 39.37 88.9)
+		(size 39.37 31.75)
+		(exclude_from_sim no)
+		(in_bom yes)
+		(on_board yes)
+		(dnp no)
+		(fields_autoplaced yes)
+		(stroke
+			(width 0.1524)
+			(type solid)
+		)
+		(fill
+			(color 0 0 0 0)
+		)
+		(property "Sheetname" "12Vbuck"
+			(at 39.37 88.1884 0)
+			(show_name no)
+			(do_not_autoplace no)
+			(effects
+				(font
+					(size 1.27 1.27)
+				)
+				(justify left bottom)
+			)
+		)
+		(property "Sheetfile" "12Vbuck.kicad_sch"
+			(at 39.37 121.2346 0)
+			(show_name no)
+			(do_not_autoplace no)
+			(effects
+				(font
+					(size 1.27 1.27)
+				)
+				(justify left top)
+			)
+		)
+		(instances
+			(project "ProteusPowerManagment"
+				(path "/c24111dd-5300-4143-a3c3-2d963194a3cb"
+					(page "3")
+				)
+			)
+		)
+	)
+	(sheet
+		(at 39.37 142.24)
+		(size 39.37 29.21)
+		(exclude_from_sim no)
+		(in_bom yes)
+		(on_board yes)
+		(dnp no)
+		(fields_autoplaced yes)
+		(stroke
+			(width 0.1524)
+			(type solid)
+		)
+		(fill
+			(color 0 0 0 0)
+		)
+		(property "Sheetname" "5Vbuck"
+			(at 39.37 141.5284 0)
+			(show_name no)
+			(do_not_autoplace no)
+			(effects
+				(font
+					(size 1.27 1.27)
+				)
+				(justify left bottom)
+			)
+		)
+		(property "Sheetfile" "5Vbuck.kicad_sch"
+			(at 39.37 172.0346 0)
+			(show_name no)
+			(do_not_autoplace no)
+			(effects
+				(font
+					(size 1.27 1.27)
+				)
+				(justify left top)
+			)
+		)
+		(instances
+			(project "ProteusPowerManagment"
+				(path "/c24111dd-5300-4143-a3c3-2d963194a3cb"
+					(page "4")
+				)
+			)
+		)
+	)
 	(sheet_instances
 		(path "/"

Commit message: starter på sikring i nytt ark
Parts:
- added C101, C102: 470u, symbol Device:C
- added CR101, CR102: SMCJ54CA, SMCJSeries_LTF, symbol Halfdan:SMCJ54CA
Connections:
- new net: C101.2, C102.1
- new net: CR101.1, CR102.1
- new net +BATT: CR101.2
- new net GND: C101.1, C102.2, CR102.2
Other:
- sheet 12Vbuck ports: added 12VSYNC_In, 12VSYNC_Out, 12V_PGOOD, 12V_Vin, 12V_Vout; removed none
- sheet 5Vbuck ports: added 5VSYNC_In, 5VSYNC_Out, 5V_PGOOD, 5V_Vin, 5V_Vout; removed none

Commit message: starter på sikring i nytt ark
Parts:
- removed C101, C102: 470u, symbol Device:C
- removed CR101, CR102: SMCJ54CA, SMCJSeries_LTF, symbol Halfdan:SMCJ54CA
Other:
- added sheet Sikring (sikring.kicad_sch)
